File: Schematic/untitled.brd (EAGLE design)
At the start: 34.9 x 46.3 mm, 16 parts

Commit message: esProg AVR Programmer
esProg AVR Programmer
Parts:
- added R5, R6, R7, R8: 100R, adafruit:R0805
- added R9: 1K, adafruit:R0805
- R4: value 6K -> 5K
- moved R4 54.0 mm to (26.7, 28.6), flipped to the bottom, turned to 270 degrees
- moved R3 47.9 mm to (24.1, 28.6), flipped to the bottom, turned to 270 degrees
Connections:
- new net N$1: R8.1, U$2.1
- new net N$2: R7.1, U$2.5
- new net N$3: R6.1, U$2.7
- new net N$4: R5.1, U$2.9
- new net N$5: R4.2, R9.1
- net BAT: now also R9.2; no longer R4.2
- net MISO: now also R5.2; no longer U$2.9
- net MOSI: now also R8.2; no longer U$2.1
- net RESET: now also R7.2; no longer U$2.5
- net SCK: now also R6.2; no longer U$2.7
Routing:
- net N$2: track 0.00 -> 29.2 mm
- net N$1: track 0.00 -> 24.4 mm, vias 0 -> 1
- net N$3: track 0.00 -> 21.8 mm
- net N$4: track 0.00 -> 16.2 mm
- net GND: track 7.62 -> 19.4 mm, vias 1 -> 0
- net RESET: track 29.3 -> 18.0 mm
- net MOSI: track 28.7 -> 19.0 mm
- net MISO: track 13.8 -> 21.1 mm, vias 0 -> 1
- net SCK: track 31.7 -> 24.6 mm, vias 2 -> 0
- net ADC: track 0.00 -> 5.99 mm
- net N$5: track 0.00 -> 2.45 mm
- net 3.3V: track 57.1 -> 55.3 mm, vias 1 -> 0
Other:
- board size 34.9 x 46.3 mm -> 49.5 x 46.3 mm
